Commit message: feat: add ArUco forward marker URDF and debugging scripts for drone kinematics and simulation logs.

File: helionv4.urdf (robot description, URDF)
Before this commit: robot helion_v4_pro, 1 links, 0 joints
Links:
- link base_link: geometry collision box size=0.34 0.34 0.063; visual box size=0.15 0.15 0.05
